File: pcb/analog/analog.kicad_sch (KiCad schematic)
At the start: 65 parts, among them J1 USB_C_Receptacle_USB2.0, SW1 SW_Push, SW2 SW_Push, U1 SRV05-4, U2 XC6206P332MR, U3 DRV5056A3xDBZxQ1, U4 DRV5056A3xDBZxQ1, U5 DRV5056A3xDBZxQ1, U6 74AHCT1G125, U7 74AHCT1G125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

Commit message: fix: ensure that mounting holes are excluded from bom
Parts:
- H1, H2, H3, H4: now left out of the parts list
Changed lines of the file:
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@@
   )
   (symbol (lib_id "Mechanical:MountingHole") (at 198.12 172.72 0) (unit 1)
-    (in_bom yes) (on_board yes) (dnp no) (fields_autoplaced)
+    (in_bom no) (on_board yes) (dnp no) (fields_autoplaced)
     (property "Reference" "H2" (at 200.66 171.45 0)
       (effects (font (size 1.27 1.27)) (justify left))
@@
   )
   (symbol (lib_id "Mechanical:MountingHole") (at 218.44 172.72 0) (unit 1)
-    (in_bom yes) (on_board yes) (dnp no) (fields_autoplaced)
+    (in_bom no) (on_board yes) (dnp no) (fields_autoplaced)
     (property "Reference" "H3" (at 220.98 171.45 0)
       (effects (font (size 1.27 1.27)) (justify left))
@@
   )
   (symbol (lib_id "Mechanical:MountingHole") (at 177.8 172.72 0) (unit 1)
-    (in_bom yes) (on_board yes) (dnp no)
+    (in_bom no) (on_board yes) (dnp no)
     (property "Reference" "H1" (at 180.34 171.45 0)
       (effects (font (size 1.27 1.27)) (justify left))
@@
   )
   (symbol (lib_id "Mechanical:MountingHole") (at 238.76 172.72 0) (unit 1)
-    (in_bom yes) (on_board yes) (dnp no) (fields_autoplaced)
+    (in_bom no) (on_board yes) (dnp no) (fields_autoplaced)
     (property "Reference" "H4" (at 241.3 171.45 0)
       (effects (font (size 1.27 1.27)) (justify left))
