File: pcb/minoripad/minoripad.kicad_sch (KiCad schematic)
At the start: 42 parts, among them J1 USB_C_Receptacle_USB2.0, SW1 SW_Push, SW2 SW_Push, U1 SRV05-4, U2 XC6206P332MR, U8 RP2040, U9 W25Q16JVSSIQ, Y1 12MHz

Commit message: fix: correct title in minoripad schematic
Other:
- title: Haruka (Analog PCB ver.) -> Minoripad
Changed lines of the file:
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@@
   (paper "A4")
   (title_block
-    (title "Haruka (Analog PCB ver.)")
+    (title "Minoripad")
     (rev "1")
   )
