File: pcb/harukapad/harukapad.kicad_pcb (KiCad board)
At the start: 2 copper layers, 70 x 70 mm, 65 parts, among them J1 USB_C_Receptacle_USB2.0, SW1 SW_Push, SW2 SW_Push, U1 SRV05-4, U2 XC6206P332MR, U3 DRV5056A4xDBZxQ1, U4 DRV5056A4xDBZxQ1, U5 DRV5056A4xDBZxQ1, U6 74AHCT1G125, U7 74AHCT1G125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

Commit message: fix(harukapad): connect mounting holes to ground, fix incorrect footprint
at some point, it changed back to the SOT-23 footprint, so the holes would've been missing...
Parts:
- U3, U4, U5: footprint Package_TO_SOT_SMD:SOT-23 -> Custom:KS-20-1U-DRV5056
- turned U3 to 180 degrees
- turned U4 to 180 degrees
- turned U5 to 180 degrees
Connections:
- H1 pad 1: (no net) -> GND
- H2 pad 1: (no net) -> GND
- H3 pad 1: (no net) -> GND
- H4 pad 1: (no net) -> GND
