File: rev1/cloverpad-mx-pcb/cloverpad-mx.kicad_sch (KiCad schematic)
At the start: 42 parts, among them J1 USB_C_Receptacle_USB2.0, SW1 SW_Push, SW2 SW_Push, U1 SRV05-4, U2 XC6206P332MR, U8 RP2040, U9 W25Q16JVSSIQ, Y1 12MHz

Commit message: chore: update all symbols + footprints to match kicad 8
Parts:
- J1: symbol Connector:USB_C_Receptacle_USB2.0 -> Connector:USB_C_Receptacle_USB2.0_16P
- MX1, MX2, MX3: footprint PCM_marbastlib-mx:SW_MX_HS_1u -> PCM_marbastlib-mx:SW_MX_HS_CPG151101S11_1u; symbol PCM_marbastlib-mx:MX_SW_HS -> PCM_marbastlib-mx:MX_SW_HS_CPG151101S11
