File: rev1/minimal-pcb/minimal-pcb.kicad_pcb (KiCad board)
At the start: 2 copper layers, 70 x 75 mm, 8 parts, among them J1 USB_C_Receptacle_USB2.0

Commit message: chore: update all symbols + footprints to match kicad 8
Parts:
- MX1, MX2, MX3: footprint PCM_marbastlib-mx:SW_MX_HS_1u -> PCM_marbastlib-mx:SW_MX_HS_CPG151101S11_1u
Connections:
- J1 pad A1: Net-(J1-GND-PadA1) -> unconnected-(J1-GND-PadA1)_1
- J1 pad A12: Net-(J1-GND-PadA1) -> unconnected-(J1-GND-PadA1)_0
- J1 pad A4: Net-(J1-VBUS-PadA4) -> unconnected-(J1-VBUS-PadA4)_0
- J1 pad A9: Net-(J1-VBUS-PadA4) -> unconnected-(J1-VBUS-PadA4)_1
- J1 pad B1: Net-(J1-GND-PadA1) -> unconnected-(J1-GND-PadA1)
- J1 pad B12: Net-(J1-GND-PadA1) -> unconnected-(J1-GND-PadA1)_2
- J1 pad B4: Net-(J1-VBUS-PadA4) -> unconnected-(J1-VBUS-PadA4)
- J1 pad B9: Net-(J1-VBUS-PadA4) -> unconnected-(J1-VBUS-PadA4)_2
